Commit message: added surface of palm fixed transform

File: urdf/barrett_hand_mount.urdf.xacro (robot description, xacro)
@@ -68,4 +68,19 @@
 	<child link="${prefix}barrett_mount_link"/>
       </joint>
+      <link name="${prefix}barrett_palm_surface_frame">
+	<inertial>
+	  <origin xyz="0 0 0" />
+	  <mass value="0.50573"/>
+	  <inertia
+	      ixx="0.0001" ixy="0.0"    ixz="0.0"
+	      iyy="0.0001" iyz="0.0"
+              izz="0.001"/>
+	</inertial>
+      </link>
+      <joint name="${prefix}barrett_palm_surface_joint" type="fixed">
+	<origin xyz="${palm_xyz_offset}" rpy="${palm_rpy_offset}"/>
+	<parent link="${parent}"/>
+	<child link="${prefix}barrett_palm_surface_frame"/>
+      </joint>
   </xacro:macro>
 </robot>

Commit message: changed barrett_palm_surface_joint to approach_tran

File: urdf/barrett_hand_mount.urdf.xacro (robot description, xacro)
@@ -68,5 +68,5 @@
 	<child link="${prefix}barrett_mount_link"/>
       </joint>
-      <link name="${prefix}barrett_palm_surface_frame">
+      <link name="${prefix}approach_tran">
 	<inertial>
 	  <origin xyz="0 0 0" />
@@ -78,8 +78,8 @@
 	</inertial>
       </link>
-      <joint name="${prefix}barrett_palm_surface_joint" type="fixed">
+      <joint name="${prefix}approach_tran_joint" type="fixed">
 	<origin xyz="${palm_xyz_offset}" rpy="${palm_rpy_offset}"/>
 	<parent link="${parent}"/>
-	<child link="${prefix}barrett_palm_surface_frame"/>
+	<child link="${prefix}approach_tran"/>
       </joint>
   </xacro:macro>

Commit message: approach tra is a fake link, so it shouldn't really have a mass

File: urdf/barrett_hand_mount.urdf.xacro (robot description, xacro)
@@ -71,5 +71,5 @@
 	<inertial>
 	  <origin xyz="0 0 0" />
-	  <mass value="0.50573"/>
+	  <mass value="0.001"/>
 	  <inertia
 	      ixx="0.0001" ixy="0.0"    ixz="0.0"
