Commit message: added surface of palm offset

File: config/arm_to_hand_calib.xacro (robot description, xacro)
@@ -1,5 +1,7 @@
 <?xml version="1.0"?>
 <robot xmlns:xacro="http://ros.org/wiki/xacro" name="arm_to_hand_calib">
-  <xacro:property name="hand_xyz_offset" value="0 0 0.0775"/>
+  <xacro:property name="hand_xyz_offset" value="0 0 0.0705"/>
   <xacro:property name="hand_rpy_offset" value="0 0 5.0614"/>
+  <xacro:property name="palm_xyz_offset" value="0 0 0.149"/>
+  <xacro:property name="palm_rpy_offset" value="0 0 1.9224"/>
 </robot>

Commit message: Fixed incorrect hand rotation

File: config/arm_to_hand_calib.xacro (robot description, xacro)
@@ -2,5 +2,6 @@
 <robot xmlns:xacro="http://ros.org/wiki/xacro" name="arm_to_hand_calib">
   <xacro:property name="hand_xyz_offset" value="0 0 0.0705"/>
-  <xacro:property name="hand_rpy_offset" value="0 0 5.0614"/>
+<!--  <xacro:property name="hand_rpy_offset" value="0 0 5.0614"/> -->
+  <xacro:property name="hand_rpy_offset" value="0 0 1.919807"/>
   <xacro:property name="palm_xyz_offset" value="0 0 0.149"/>
   <xacro:property name="palm_rpy_offset" value="0 0 1.9224"/>

Commit message: changed the reference file for barrett hand

File: config/arm_to_hand_calib.xacro (robot description, xacro)
@@ -2,7 +2,8 @@
 <robot xmlns:xacro="http://ros.org/wiki/xacro" name="arm_to_hand_calib">
   <xacro:property name="hand_xyz_offset" value="0 0 0.0705"/>
-<!--  <xacro:property name="hand_rpy_offset" value="0 0 5.0614"/> -->
-  <xacro:property name="hand_rpy_offset" value="0 0 1.919807"/>
+  <xacro:property name="hand_rpy_offset" value="0 0 5.0614"/>
+  <!--<xacro:property name="hand_rpy_offset" value="0 0 1.919807"/> -->
   <xacro:property name="palm_xyz_offset" value="0 0 0.149"/>
-  <xacro:property name="palm_rpy_offset" value="0 0 1.9224"/>
+  <!--<xacro:property name="palm_rpy_offset" value="0 0 1.9224"/>-->
+  <xacro:property name="palm_rpy_offset" value="0 0 5.0614"/>
 </robot>

File: urdf/staubli_bhand.xacro (robot description, xacro)
@@ -6,5 +6,5 @@
 <xacro:include filename="$(find staubli_description)/urdf/tx60l_macro.xacro"/>
  <!-- Include Barrett Hand robot -->
-<xacro:include filename="$(find barrett_hand_description)/urdf/bh282.urdf.xacro" />
+<xacro:include filename="$(find barrett_hand_description)/urdf/bh280.urdf.xacro" />
 <!-- Include the barrett hands mount on the staubli -->
 <xacro:include filename="$(find staubli_barretthand_description)/urdf/barrett_hand_mount.urdf.xacro"/>
